File: Electronics/V1/V1.kicad_sch (KiCad schematic)
At the start: 0 parts

Commit message: Added USB port to schematic
Parts:
- added J1: USB_C_Receptacle_USB2.0_16P, symbol Connector:USB_C_Receptacle_USB2.0_16P
- added R1, R2: 5k1, symbol Device:R_Small
- added U1: RP2350A, Package_DFN_QFN:QFN-60-1EP_7x7mm_P0.4mm_EP3.4x3.4mm, symbol MCU_RaspberryPi:RP2350A
Connections:
- new net: U1.1 (IOVDD), U1.11 (IOVDD), U1.20 (IOVDD), U1.30 (IOVDD), U1.38 (IOVDD), U1.45 (IOVDD)
- new net: U1.23 (DVDD), U1.39 (DVDD), U1.6 (DVDD)
- new net: J1.A5 (CC1), R1.1
- new net: J1.B5 (CC2), R2.1
- new net +3V3: J1.A4 (VBUS), J1.A9 (VBUS), J1.B4 (VBUS), J1.B9 (VBUS)
- new net DATA+: J1.A7 (D-), J1.B7 (D-), U1.52 (USB_DP)
- new net DATA-: J1.A6 (D+), J1.B6 (D+), U1.51 (USB_DM)
- new net GND: J1.A1 (GND), J1.A12 (GND), J1.B1 (GND), J1.B12 (GND), J1.SH (SHIELD), R1.2, R2.2
- no-connect marks 0 -> 2

Commit message: added crystal circuit and fixed usb stuff i messed up earlier
Parts:
- added C1, C2: 22p, symbol Device:C_Small
- added F1: Fuse_Small, symbol Device:Fuse_Small
- added R3: 1k, symbol Device:R_Small
- added R4, R5: 27, symbol Device:R_Small
- added U2: SRV05-4, Package_TO_SOT_SMD:SOT-23-6, symbol Power_Protection:SRV05-4
- added Y1: Crystal_GND24, symbol XIAO_RP2040:Crystal_GND24
Connections:
- net DATA+: now also R4.2, U2.1 (IO1); no longer U1.52 (USB_DP)
- net DATA-: now also R5.2, U2.3 (IO2); no longer U1.51 (USB_DM)
- net GND: now also C1.1, C2.1, U2.2 (VN), Y1.2 (G), Y1.4 (G)
- net XIN: now reaches U1.21 (XIN)
- net XIN: now also C1.2, Y1.3
- net XOUT: now reaches U1.22 (XOUT)
- net XOUT: now also R3.1
- net +3V3 renamed VBUS
- net VBUS: now also F1.1
- new net: R5.1, U1.51 (USB_DM)
- new net: C2.2, R3.2, Y1.1
- new net: R4.1, U1.52 (USB_DP)
- new net +5V: F1.2, U2.5 (VP)
- no-connect marks 2 -> 4
